Commit message: update v1

File: urdf/husky/husky.urdf (robot description, URDF)
Before this commit: robot husky_robot, 11 links, 10 joints
Joints:
- joint front_left_wheel: limit (none) -> effort=100.0 velocity=10.0
- joint front_right_wheel: limit (none) -> effort=100.0 velocity=10.0
- joint imu_joint: origin xyz=$(optenv HUSKY_IMU_XYZ 0.19 0 0.149) rpy=$(optenv HUSKY_IMU_RPY 0 -1.5708 3.1416) -> xyz=0.19 0 0.149 rpy=0 -1.5708 3.1416
- joint rear_left_wheel: limit (none) -> effort=100.0 velocity=10.0
- joint rear_right_wheel: limit (none) -> effort=100.0 velocity=10.0
